File: rj45_ports.sch (KiCad schematic (older format))
At the start: 24 parts, among them J2201 BEL_0845_2G1T_H5, U2201 74LVC1G06, U2202 74LVC1G06

Commit message: added more component values/part numbers
Parts:
- FB2201: Manufacturer (none) -> TDK
- J2201: Manufacturer (none) -> BEL; Part (none) -> 0845-2G1T-H5
Changed lines of the file:
@@
 F 2 "proj_footprints:BEL_0845-2G1T-H5" H 5400 1550 50  0001 C CNN
 F 3 "https://www.mouser.ch/datasheet/2/643/dr-MAG-0845-2G1T-H5-1309698.pdf" H 4985 2065 50  0001 L TNN
+F 4 "0845-2G1T-H5" H 5400 2300 50  0001 C CNN "Part"
+F 5 "BEL" H 5400 2300 50  0001 C CNN "Manufacturer"
 	1    5400 2300
 	-1   0    0    -1
@@
 F 3 "~" H 7150 3800 50  0001 C CNN
 F 4 "MPZ1608S221ATA00" H 7150 3800 50  0001 C CNN "Part"
+F 5 "TDK" H 7150 3800 50  0001 C CNN "Manufacturer"
 	1    7150 3800
 	1    0    0    -1

Commit message: some fixes; don't recall details :-(
Parts:
- U2201, U2202: footprint Package_TO_SOT_SMD:SOT-553 -> proj_footprints:SOT-5x3
Changed lines of the file:
@@
 F 0 "U2201" H 4650 1600 50  0000 L CNN
 F 1 "74LVC1G06" H 4300 1450 50  0000 L CNN
-F 2 "Package_TO_SOT_SMD:SOT-553" H 4900 1350 50  0001 C CNN
+F 2 "proj_footprints:SOT-5x3" H 4900 1350 50  0001 C CNN
 F 3 "http://www.ti.com/lit/sg/scyt129e/scyt129e.pdf" H 4900 1350 50  0001 C CNN
 	1    4900 1350
@@
 F 0 "U2202" H 4650 3800 50  0000 L CNN
 F 1 "74LVC1G06" H 4300 3650 50  0000 L CNN
-F 2 "Package_TO_SOT_SMD:SOT-553" H 4900 3550 50  0001 C CNN
+F 2 "proj_footprints:SOT-5x3" H 4900 3550 50  0001 C CNN
 F 3 "http://www.ti.com/lit/sg/scyt129e/scyt129e.pdf" H 4900 3550 50  0001 C CNN
 	1    4900 3550

Commit message: WIP save
Parts:
- removed U2201: 74LVC1G06, proj_footprints:SOT-5x3, symbol fmc:74LVC1G06
- added JP2201: 100FDb, Connector_PinHeader_2.54mm:PinHeader_1x03_P2.54mm_Vertical, symbol Jumper:Jumper_3_Bridged12
- added R2211: 100, Resistor_SMD:R_0603_1608Metric, symbol Device:R_Small
- added U2201: 74AHC1T86, Package_TO_SOT_SMD:SOT-353_SC-70-5, symbol fmc:74AHC1G86
Connections:
- wire segments 103 -> 112
Other:
- note added: "Level-translating gate!"
- moved on the sheet: R2209
Changed lines of the file:
@@
 $Descr A4 11693 8268
 encoding utf-8
-Sheet 8 12
+Sheet 5 18
 Title ""
 Date ""
@@
 	1    0    0    -1
 $EndComp
-$Comp
-L Device:R_Small R2209
-U 1 1 60E01790
-P 5350 1350
-F 0 "R2209" H 5409 1396 50  0000 L CNN
-F 1 "100" H 5409 1305 50  0000 L CNN
-F 2 "Resistor_SMD:R_0603_1608Metric" H 5350 1350 50  0001 C CNN
-F 3 "~" H 5350 1350 50  0001 C CNN
-	1    5350 1350
-	0    1    1    0
-$EndComp
-$Comp
-L lan9254_project:+3V3 #PWR?
-U 1 1 60E04837
-P 5600 1100
-F 0 "#PWR?" H 5600 950 50  0001 C CNN
-F 1 "+3V3" H 5615 1273 50  0000 C CNN
-F 2 "" H 5600 1100 50  0001 C CNN
-F 3 "" H 5600 1100 50  0001 C CNN
-	1    5600 1100
-	1    0    0    -1
-$EndComp
 Text HLabel 1750 1350 0    50   Input ~ 0
 P0_ACTLED
@@
 F 3 "" H 4900 1550 50  0001 C CNN
 	1    4900 1550
-	1    0    0    -1
-$EndComp
-$Comp
-L lan9254_project:+1V8 #PWR?
-U 1 1 60E6480F
-P 4900 1150
-F 0 "#PWR?" H 4900 1000 50  0001 C CNN
-F 1 "+1V8" H 4915 1323 50  0000 C CNN
-F 2 "" H 4900 1150 50  0001 C CNN
-F 3 "" H 4900 1150 50  0001 C CNN
-	1    4900 1150
 	1    0    0    -1
 $EndComp
@@
 	7150 3550 7150 3700
 Connection ~ 7150 3700
-$Comp
-L fmc:74LVC1G06 U2201
-U 1 1 61143898
-P 4900 1350
-F 0 "U2201" H 4650 1600 50  0000 L CNN
-F 1 "74LVC1G06" H 4300 1450 50  0000 L CNN
-F 2 "proj_footprints:SOT-5x3" H 4900 1350 50  0001 C CNN
-F 3 "http://www.ti.com/lit/sg/scyt129e/scyt129e.pdf" H 4900 1350 50  0001 C CNN
-	1    4900 1350
-	1    0    0    -1
-$EndComp
-Wire Wire Line
-	1750 1350 4600 1350
+Wire Wire Line
+	1750 1350 3600 1350
 $Comp
 L lan9254_project:GND #PWR?
@@
 	1750 3550 4600 3550
 Wire Wire Line
-	5600 1100 5600 1700
-Wire Wire Line
-	5450 1350 5500 1350
-Wire Wire Line
-	5500 1350 5500 1700
-Wire Wire Line
-	5150 1350 5250 1350
-Wire Wire Line
 	5600 3300 5600 3900
 Wire Wire Line
@@
 Wire Wire Line
 	5250 3550 5150 3550
+$Comp
+L fmc:74AHC1G86 U2201
+U 1 1 61F876C4
+P 4900 1300
+F 0 "U2201" H 4800 1800 50  0000 L CNN
+F 1 "74AHC1T86" H 4800 1900 50  0000 L CNN
+F 2 "Package_TO_SOT_SMD:SOT-353_SC-70-5" H 4900 1300 50  0001 C CNN
+F 3 "http://www.ti.com/lit/sg/scyt129e/scyt129e.pdf" H 4900 1300 50  0001 C CNN
+	1    4900 1300
+	1    0    0    -1
+$EndComp
+$Comp
+L lan9254_project:+3V3 #PWR?
+U 1 1 60E04837
+P 4900 1100
+F 0 "#PWR?" H 4900 950 50  0001 C CNN
+F 1 "+3V3" H 4915 1273 50  0000 C CNN
+F 2 "" H 4900 1100 50  0001 C CNN
+F 3 "" H 4900 1100 50  0001 C CNN
+	1    4900 1100
+	1    0    0    -1
+$EndComp
+$Comp
+L Device:R_Small R2209
+U 1 1 60E01790
+P 5350 1300
+F 0 "R2209" H 5000 1350 50  0000 L CNN
+F 1 "100" H 5100 1250 50  0000 L CNN
+F 2 "Resistor_SMD:R_0603_1608Metric" H 5350 1300 50  0001 C CNN
+F 3 "~" H 5350 1300 50  0001 C CNN
+	1    5350 1300
+	0    1    1    0
+$EndComp
+Wire Wire Line
+	5150 1300 5250 1300
+Wire Wire Line
+	4900 1500 4900 1550
+Wire Wire Line
+	5450 1300 5600 1300
+Wire Wire Line
+	5600 1300 5600 1700
+Wire Wire Line
+	5500 1700 5500 1500
+Wire Wire Line
+	5500 1500 4900 1500
+Connection ~ 4900 1500
+Text Notes 4750 600  0    50   ~ 0
+Level-translating gate!
+$Comp
+L Jumper:Jumper_3_Bridged12 JP2201
+U 1 1 61FA3E41
+P 4300 1100
+F 0 "JP2201" H 4300 1304 50  0000 C CNN
+F 1 "100FDb" H 4300 1213 50  0000 C CNN
+F 2 "Connector_PinHeader_2.54mm:PinHeader_1x03_P2.54mm_Vertical" H 4300 1100 50  0001 C CNN
+F 3 "~" H 4300 1100 50  0001 C CNN
+	1    4300 1100
+	-1   0    0    -1
+$EndComp
+Wire Wire Line
+	4300 1250 4600 1250
+$Comp
+L Device:R_Small R2211
+U 1 1 61FAC493
+P 3800 1250
+F 0 "R2211" H 3500 1300 50  0000 L CNN
+F 1 "100" H 3550 1200 50  0000 L CNN
+F 2 "Resistor_SMD:R_0603_1608Metric" H 3800 1250 50  0001 C CNN
+F 3 "~" H 3800 1250 50  0001 C CNN
+	1    3800 1250
+	0    1    1    0
+$EndComp
+$Comp
+L lan9254_project:+1V8 #PWR?
+U 1 1 61FACEB2
+P 4550 1100
+F 0 "#PWR?" H 4550 950 50  0001 C CNN
+F 1 "+1V8" H 4565 1273 50  0000 C CNN
+F 2 "" H 4550 1100 50  0001 C CNN
+F 3 "" H 4550 1100 50  0001 C CNN
+	1    4550 1100
+	1    0    0    -1
+$EndComp
+Wire Wire Line
+	3900 1250 4300 1250
+Connection ~ 4300 1250
+Wire Wire Line
+	3700 1250 3600 1250
+Wire Wire Line
+	3600 1250 3600 1350
+Connection ~ 3600 1350
+Wire Wire Line
+	3600 1350 4600 1350
+Wire Wire Line
+	4050 1100 4050 1500
+Wire Wire Line
+	4050 1500 4900 1500
 $EndSCHEMATC

Commit message: further work...
Parts:
- R2209, R2210: value 100 -> 178
- R2211: value 100 -> 10k
- U2202: footprint proj_footprints:SOT-5x3 -> Package_TO_SOT_SMD:SOT-353_SC-70-5; symbol fmc:74LVC1G06 -> fmc:74LVC1G38
Connections:
- wire segments 112 -> 114
Changed lines of the file:
@@
 $Descr A4 11693 8268
 encoding utf-8
-Sheet 14 18
+Sheet 13 20
 Title ""
 Date ""
@@
 P 5350 3550
 F 0 "R2210" H 5409 3596 50  0000 L CNN
-F 1 "100" H 5409 3505 50  0000 L CNN
+F 1 "178" H 5409 3505 50  0000 L CNN
 F 2 "Resistor_SMD:R_0603_1608Metric" H 5350 3550 50  0001 C CNN
 F 3 "~" H 5350 3550 50  0001 C CNN
@@
 $EndComp
 $Comp
-L fmc:74LVC1G06 U2202
+L fmc:74LVC1G38 U2202
 U 1 1 61157A24
 P 4900 3550
 F 0 "U2202" H 4650 3800 50  0000 L CNN
 F 1 "74LVC1G06" H 4300 3650 50  0000 L CNN
-F 2 "proj_footprints:SOT-5x3" H 4900 3550 50  0001 C CNN
+F 2 "Package_TO_SOT_SMD:SOT-353_SC-70-5" H 4900 3550 50  0001 C CNN
 F 3 "http://www.ti.com/lit/sg/scyt129e/scyt129e.pdf" H 4900 3550 50  0001 C CNN
 	1    4900 3550
@@
 P 5350 1300
 F 0 "R2209" H 5000 1350 50  0000 L CNN
-F 1 "100" H 5100 1250 50  0000 L CNN
+F 1 "178" H 5100 1250 50  0000 L CNN
 F 2 "Resistor_SMD:R_0603_1608Metric" H 5350 1300 50  0001 C CNN
 F 3 "~" H 5350 1300 50  0001 C CNN
@@
 P 3800 1250
 F 0 "R2211" H 3500 1300 50  0000 L CNN
-F 1 "100" H 3550 1200 50  0000 L CNN
+F 1 "10k" H 3550 1200 50  0000 L CNN
 F 2 "Resistor_SMD:R_0603_1608Metric" H 3800 1250 50  0001 C CNN
 F 3 "~" H 3800 1250 50  0001 C CNN
@@
 Wire Wire Line
 	4050 1500 4900 1500
+Wire Wire Line
+	4600 3500 4600 3550
+Connection ~ 4600 3550
+Wire Wire Line
+	4600 3550 4600 3600
 $EndSCHEMATC
