File: strap.sch (KiCad schematic (older format))
At the start: 20 parts, among them SW2101 SW_DIP_x08, U2101 74LVC1G06, U2102 74LVC1G06, U2103 PCA9306, U2104 24AA0x

Commit message: fixed i2c switch (Vref2 is *not* a normal power input); small fixes
Parts:
- added C2101, C2103: 100n, Capacitor_SMD:C_0402_1005Metric, symbol Device:C_Small
- added C2102: 100p, Capacitor_SMD:C_0402_1005Metric, symbol Device:C_Small
- added R2113: 100k, Resistor_SMD:R_0603_1608Metric, symbol Device:R_Small
- D2101: value LED_Small -> LED; symbol Device:LED_Small -> Device:LED; Manufacturer (none) -> Wurth; Part (none) -> 150060RS75000
- D2102: value LED_Small -> LED; symbol Device:LED_Small -> Device:LED; Manufacturer (none) -> Wurth; Part (none) -> 150060GS75000
- R18, R19: value 10k -> 3k3
- R23: value 4k7 -> 5k1
- R26: value 10k -> 100k
Connections:
- wire segments 94 -> 105
Other:
- moved on the sheet: R2112, U2104

Commit message: some fixes; don't recall details :-(
Parts:
- U2101, U2102: footprint Package_TO_SOT_SMD:SOT-553 -> proj_footprints:SOT-5x3
Changed lines of the file:
@@
 F 0 "U2101" H 4550 5300 50  0000 L CNN
 F 1 "74LVC1G06" H 4400 4900 50  0000 L CNN
-F 2 "Package_TO_SOT_SMD:SOT-553" H 4900 5100 50  0001 C CNN
+F 2 "proj_footprints:SOT-5x3" H 4900 5100 50  0001 C CNN
 F 3 "http://www.ti.com/lit/sg/scyt129e/scyt129e.pdf" H 4900 5100 50  0001 C CNN
 	1    4900 5100
@@
 F 0 "U2102" H 4550 6500 50  0000 L CNN
 F 1 "74LVC1G06" H 4400 6100 50  0000 L CNN
-F 2 "Package_TO_SOT_SMD:SOT-553" H 4900 6300 50  0001 C CNN
+F 2 "proj_footprints:SOT-5x3" H 4900 6300 50  0001 C CNN
 F 3 "http://www.ti.com/lit/sg/scyt129e/scyt129e.pdf" H 4900 6300 50  0001 C CNN
 	1    4900 6300

Commit message: WIP save
Parts:
- removed R21: 1k, Resistor_SMD:R_0603_1608Metric, symbol Device:R_Small
- removed U2101, U2102: 74LVC1G06, proj_footprints:SOT-5x3, symbol fmc:74LVC1G06
- added R2107, R2114: 100k, Resistor_SMD:R_0603_1608Metric, symbol Device:R_Small
- added U2101, U2102, U2105, U2106: 74AHC1T86, Package_TO_SOT_SMD:SOT-353_SC-70-5, symbol fmc:74AHC1G86
Connections:
- wire segments 105 -> 127
- no-connect marks 6 -> 9
Other:
- note added: "For routing reasons this is now\na dedicated jumper elsewhere!"
- note added: "T-version: Level-translating gate!"
- moved on the sheet: R2106, R2108, R2109

Commit message: changed LED drivers; added Jumpers, write-protect
Modified LED drivers (XOR approach) to work with lan9254's
open-drain/-source outputs.

Routed spare switches as jumpers out of this module.

Route eeprom-write protect out of this module.
Route eeprom-isolation switch info out (so that FPGA may easily
determine whether EEPROM emulation is used or not).
Parts:
- added R2115: 10k, Resistor_SMD:R_0603_1608Metric, symbol Device:R_Small
Connections:
- net labels added: EEP_SZ, EEP_WP, I2C_ISOLb, JP7, JP8, SCL, SDA
- net labels removed: SCL_3V3, SDA_3V3
- wire segments 127 -> 141
- no-connect marks 9 -> 5
Other:
- moved on the sheet: R2101, R2102
Changed lines of the file:
@@
 $Descr A4 11693 8268
 encoding utf-8
-Sheet 6 18
+Sheet 15 18
 Title ""
 Date ""
@@
 Text HLabel 3800 3000 0    50   BiDi ~ 0
 RUNLED#EE_EMUL0
-Text HLabel 3800 1300 0    50   BiDi ~ 0
+Text HLabel 3800 1500 0    50   BiDi ~ 0
 XTAL_MODE
 Text HLabel 3800 3650 0    50   BiDi ~ 0
@@
 EE_EMUL_SPI0
 NoConn ~ 3800 3750
-Text Notes 3100 1250 0    50   ~ 0
+Text Notes 3100 1450 0    50   ~ 0
 VDD3V3 (analog)\n
 $Comp
@@
 Text Notes 3850 2200 0    50   ~ 0
 (PU)
-Text Notes 3850 1300 0    50   ~ 0
+Text Notes 3850 1500 0    50   ~ 0
 (mid)
 Text Notes 3850 3650 0    50   ~ 0
@@
 L Device:R_Small R?
 U 1 1 60E7CBCF
-P 4150 1300
+P 4150 1500
 AR Path="/60DC28BD/60E7CBCF" Ref="R?"  Part="1"
 AR Path="/60E5E32B/60E7CBCF" Ref="R14"  Part="1"
 AR Path="/60DB2574/60E5E32B/60E7CBCF" Ref="R2101"  Part="1"
 AR Path="/60E70F2C/60E5E32B/60E7CBCF" Ref="R2101"  Part="1"
-F 0 "R2101" V 4250 1050 50  0000 C CNN
-F 1 "1k" V 4255 1300 50  0000 C CNN
-F 2 "Resistor_SMD:R_0603_1608Metric" H 4150 1300 50  0001 C CNN
-F 3 "~" H 4150 1300 50  0001 C CNN
-	1    4150 1300
+F 0 "R2101" V 4250 1250 50  0000 C CNN
+F 1 "1k" V 4255 1500 50  0000 C CNN
+F 2 "Resistor_SMD:R_0603_1608Metric" H 4150 1500 50  0001 C CNN
+F 3 "~" H 4150 1500 50  0001 C CNN
+	1    4150 1500
 	0    -1   -1   0
 $EndComp
@@
 L lan9254_project:GND #PWR?
 U 1 1 60E7CC6D
-P 4400 1300
+P 4400 1500
 AR Path="/60DC28BD/60E7CC6D" Ref="#PWR?"  Part="1"
 AR Path="/60E5E32B/60E7CC6D" Ref="#PWR?"  Part="1"
 AR Path="/60DB2574/60E5E32B/60E7CC6D" Ref="#PWR?"  Part="1"
 AR Path="/60E70F2C/60E5E32B/60E7CC6D" Ref="#PWR?"  Part="1"
-F 0 "#PWR?" H 4400 1050 50  0001 C CNN
-F 1 "GND" V 4405 1172 50  0000 R CNN
-F 2 "" H 4400 1300 50  0001 C CNN
-F 3 "" H 4400 1300 50  0001 C CNN
-	1    4400 1300
+F 0 "#PWR?" H 4400 1250 50  0001 C CNN
+F 1 "GND" V 4405 1372 50  0000 R CNN
+F 2 "" H 4400 1500 50  0001 C CNN
+F 3 "" H 4400 1500 50  0001 C CNN
+	1    4400 1500
 	0    -1   -1   0
 $EndComp
 Wire Wire Line
-	4250 1300 4400 1300
-Wire Wire Line
-	4050 1300 3900 1300
+	4250 1500 4400 1500
+Wire Wire Line
+	4050 1500 3900 1500
 Text Notes 3850 3100 0    50   ~ 0
 (PU)
@@
 	6300 4400 6350 4400
 Text HLabel 10300 2800 2    50   BiDi ~ 0
-SCL_3V3
+SCL
 Text HLabel 10300 2900 2    50   BiDi ~ 0
-SDA_3V3
+SDA
 Wire Wire Line
 	4450 3000 4500 3000
@@
 L Device:R_Small R?
 U 1 1 60DB9030
-P 4150 1550
+P 4150 1750
 AR Path="/60DC28BD/60DB9030" Ref="R?"  Part="1"
 AR Path="/60E5E32B/60DB9030" Ref="R15"  Part="1"
 AR Path="/60DB2574/60E5E32B/60DB9030" Ref="R2102"  Part="1"
 AR Path="/60E70F2C/60E5E32B/60DB9030" Ref="R2102"  Part="1"
-F 0 "R2102" V 4250 1300 50  0000 C CNN
-F 1 "1k" V 4255 1550 50  0000 C CNN
-F 2 "Resistor_SMD:R_0603_1608Metric" H 4150 1550 50  0001 C CNN
-F 3 "~" H 4150 1550 50  0001 C CNN
-	1    4150 1550
+F 0 "R2102" V 4250 1500 50  0000 C CNN
+F 1 "1k" V 4255 1750 50  0000 C CNN
+F 2 "Resistor_SMD:R_0603_1608Metric" H 4150 1750 50  0001 C CNN
+F 3 "~" H 4150 1750 50  0001 C CNN
+	1    4150 1750
 	0    -1   -1   0
 $EndComp
@@
 L lan9254_project:+3V3 #PWR?
 U 1 1 60DB9387
-P 4400 1550
+P 4400 1750
 AR Path="/60DC28BD/60DB9387" Ref="#PWR?"  Part="1"
 AR Path="/60E5E32B/60DB9387" Ref="#PWR?"  Part="1"
 AR Path="/60DB2574/60E5E32B/60DB9387" Ref="#PWR?"  Part="1"
 AR Path="/60E70F2C/60E5E32B/60DB9387" Ref="#PWR?"  Part="1"
-F 0 "#PWR?" H 4400 1400 50  0001 C CNN
-F 1 "+3V3" H 4415 1723 50  0000 C CNN
-F 2 "" H 4400 1550 50  0001 C CNN
-F 3 "" H 4400 1550 50  0001 C CNN
-	1    4400 1550
+F 0 "#PWR?" H 4400 1600 50  0001 C CNN
+F 1 "+3V3" H 4415 1923 50  0000 C CNN
+F 2 "" H 4400 1750 50  0001 C CNN
+F 3 "" H 4400 1750 50  0001 C CNN
+	1    4400 1750
 	0    1    1    0
 $EndComp
 Wire Wire Line
-	4400 1550 4250 1550
-Wire Wire Line
-	4050 1550 3900 1550
-Wire Wire Line
-	3900 1550 3900 1300
-Connection ~ 3900 1300
-Wire Wire Line
-	3900 1300 3800 1300
+	4400 1750 4250 1750
+Wire Wire Line
+	4050 1750 3900 1750
+Wire Wire Line
+	3900 1750 3900 1500
+Connection ~ 3900 1500
+Wire Wire Line
+	3900 1500 3800 1500
 Wire Wire Line
 	3800 7100 4050 7100
-Text HLabel 9600 2200 2    50   Input ~ 0
+Text HLabel 10300 2200 2    50   Input ~ 0
 I2C_VCC
 Wire Wire Line
@@
 Wire Wire Line
 	9650 3150 9900 3150
-Wire Wire Line
-	9900 3150 9900 3550
 $Comp
 L lan9254_project:GND #PWR?
@@
 Wire Wire Line
 	9850 3550 9900 3550
-Connection ~ 9900 3550
 Wire Wire Line
 	9900 3550 9900 4050
@@
 	5950 4400 6050 4400
 Connection ~ 6050 4400
-NoConn ~ 6650 4350
-NoConn ~ 6650 3750
 $Comp
 L Jumper:Jumper_3_Bridged12 JP2101
@@
 Connection ~ 9250 2200
 Wire Wire Line
-	9250 2200 9600 2200
+	9250 2200 10300 2200
 Wire Wire Line
 	7700 2800 9550 2800
@@
 Wire Wire Line
 	6450 3650 6450 3750
-NoConn ~ 6550 3750
-NoConn ~ 6550 4350
 $Comp
 L lan9254_project:+1V8 #PWR?
@@
 $EndComp
 Connection ~ 4900 3400
+Text HLabel 3800 700  0    50   Output ~ 0
+I2C_ISOLb
+Text HLabel 3800 850  0    50   Output ~ 0
+JP8
+Text HLabel 3800 1000 0    50   Output ~ 0
+JP7
+Wire Wire Line
+	6550 3750 6550 1000
+Wire Wire Line
+	6550 1000 3800 1000
+Wire Wire Line
+	6650 3750 6650 850
+Wire Wire Line
+	6650 850  3800 850
+Wire Wire Line
+	8650 2200 8650 700
+Wire Wire Line
+	8650 700  3800 700
+Wire Wire Line
+	6650 4350 6650 4400
+Wire Wire Line
+	6650 4400 6550 4400
+Connection ~ 6450 4400
+Wire Wire Line
+	6550 4350 6550 4400
+Connection ~ 6550 4400
+Wire Wire Line
+	6550 4400 6450 4400
+Text HLabel 10300 3150 2    50   Input ~ 0
+EEP_WP
+$Comp
+L Device:R_Small R?
+U 1 1 6202FC5D
+P 9900 3350
+AR Path="/60DC28BD/6202FC5D" Ref="R?"  Part="1"
+AR Path="/60E5E32B/6202FC5D" Ref="R?"  Part="1"
+AR Path="/60DB2574/60E5E32B/6202FC5D" Ref="R?"  Part="1"
+AR Path="/60E70F2C/60E5E32B/6202FC5D" Ref="R2115"  Part="1"
+F 0 "R2115" H 9959 3396 50  0000 L CNN
+F 1 "10k" H 9959 3305 50  0000 L CNN
+F 2 "Resistor_SMD:R_0603_1608Metric" H 9900 3350 50  0001 C CNN
+F 3 "~" H 9900 3350 50  0001 C CNN
+	1    9900 3350
+	1    0    0    -1
+$EndComp
+Wire Wire Line
+	9900 3250 9900 3150
+Connection ~ 9900 3150
+Wire Wire Line
+	9900 3150 10300 3150
+Wire Wire Line
+	9900 3450 9900 3550
+Connection ~ 9900 3550
+Wire Wire Line
+	6350 3550 6350 1150
+Connection ~ 6350 3550
+Wire Wire Line
+	3800 1150 6350 1150
+Text HLabel 3800 1150 0    50   Output ~ 0
+EEP_SZ
 $EndSCHEMATC

Commit message: further work...
Parts:
- added R2116, R2117: 0, Resistor_SMD:R_0603_1608Metric, symbol Device:R_Small
- R22: value 1k -> 10k
- R24: value 100 -> 1k5
- R25: value 100 -> 3k3
- U2104: value 24AA0x -> 24FC16T
Connections:
- wire segments 141 -> 148
Other:
- note added: "GREEN (RunLED)"
- note added: "Instead of U2105\nR2116 OR R2117\njumpers could be loaded."
- note added: "RED (ErrLED)"
- note added: "Use pin-2 input;\ncould also load\na 74LV1T04 inverter\nor a 74LV1T00 NAND"
- moved on the sheet: R2114
Changed lines of the file:
@@
 $Descr A4 11693 8268
 encoding utf-8
-Sheet 15 18
+Sheet 14 20
 Title ""
 Date ""
@@
 AR Path="/60E70F2C/60E5E32B/60E86BE2" Ref="R2108"  Part="1"
 F 0 "R2108" V 4400 2850 50  0000 C CNN
-F 1 "1k" V 4400 3150 50  0000 C CNN
+F 1 "10k" V 4400 3150 50  0000 C CNN
 F 2 "Resistor_SMD:R_0603_1608Metric" H 4350 3000 50  0001 C CNN
 F 3 "~" H 4350 3000 50  0001 C CNN
@@
 	6050 4400 6150 4400
 Wire Wire Line
-	6450 4350 6450 4400
-Wire Wire Line
-	6350 4350 6350 4400
-Connection ~ 6350 4400
-Wire Wire Line
-	6350 4400 6450 4400
-Wire Wire Line
 	6250 4350 6250 4400
 Connection ~ 6250 4400
@@
 L lan9254_project:GND #PWR?
 U 1 1 60E91F5F
-P 6300 4500
+P 6300 4550
 AR Path="/60DC28BD/60E91F5F" Ref="#PWR?"  Part="1"
 AR Path="/60E5E32B/60E91F5F" Ref="#PWR?"  Part="1"
 AR Path="/60DB2574/60E5E32B/60E91F5F" Ref="#PWR?"  Part="1"
 AR Path="/60E70F2C/60E5E32B/60E91F5F" Ref="#PWR?"  Part="1"
-F 0 "#PWR?" H 6300 4250 50  0001 C CNN
-F 1 "GND" H 6305 4327 50  0000 C CNN
-F 2 "" H 6300 4500 50  0001 C CNN
-F 3 "" H 6300 4500 50  0001 C CNN
-	1    6300 4500
-	1    0    0    -1
-$EndComp
-Wire Wire Line
-	6300 4400 6300 4500
+F 0 "#PWR?" H 6300 4300 50  0001 C CNN
+F 1 "GND" H 6305 4377 50  0000 C CNN
+F 2 "" H 6300 4550 50  0001 C CNN
+F 3 "" H 6300 4550 50  0001 C CNN
+	1    6300 4550
+	1    0    0    -1
+$EndComp
+Wire Wire Line
+	6300 4400 6300 4550
 Connection ~ 6300 4400
-Wire Wire Line
-	6300 4400 6350 4400
 Text HLabel 10300 2800 2    50   BiDi ~ 0
 SCL
@@
 AR Path="/60E70F2C/60E5E32B/60E9E985" Ref="R2110"  Part="1"
 F 0 "R2110" V 5154 5100 50  0000 C CNN
-F 1 "100" V 5245 5100 50  0000 C CNN
+F 1 "1k5" V 5245 5100 50  0000 C CNN
 F 2 "Resistor_SMD:R_0603_1608Metric" H 5350 5100 50  0001 C CNN
 F 3 "~" H 5350 5100 50  0001 C CNN
@@
 AR Path="/60E70F2C/60E5E32B/60EA51EB" Ref="R2111"  Part="1"
 F 0 "R2111" V 5154 6300 50  0000 C CNN
-F 1 "100" V 5245 6300 50  0000 C CNN
+F 1 "3k3" V 5245 6300 50  0000 C CNN
 F 2 "Resistor_SMD:R_0603_1608Metric" H 5350 6300 50  0001 C CNN
 F 3 "~" H 5350 6300 50  0001 C CNN
@@
 P 9550 3550
 F 0 "U2104" V 9175 3550 50  0000 C CNN
-F 1 "24AA0x" V 9084 3550 50  0000 C CNN
+F 1 "24FC16T" V 9084 3550 50  0000 C CNN
 F 2 "Package_TO_SOT_SMD:SOT-23-5" H 9550 3550 50  0001 C CNN
 F 3 "http://ww1.microchip.com/downloads/en/DeviceDoc/21709J.pdf" H 9550 3550 50  0001 C CNN
@@
 $EndComp
 Wire Wire Line
-	4600 5050 4600 4300
-Wire Wire Line
 	4450 3400 4600 3400
 Wire Wire Line
@@
 U 1 1 62005576
 P 4900 4300
-F 0 "U2106" H 4350 4300 50  0000 L CNN
+F 0 "U2106" H 4200 4300 50  0000 L CNN
 F 1 "74AHC1T86" H 4100 4400 50  0000 L CNN
 F 2 "Package_TO_SOT_SMD:SOT-353_SC-70-5" H 4900 4300 50  0001 C CNN
@@
 U 1 1 62010771
 P 4900 3600
-F 0 "U2105" H 4350 3600 50  0000 L CNN
+F 0 "U2105" H 4250 3600 50  0000 L CNN
 F 1 "74AHC1T86" H 4100 3700 50  0000 L CNN
 F 2 "Package_TO_SOT_SMD:SOT-353_SC-70-5" H 4900 3600 50  0001 C CNN
@@
 Connection ~ 4500 3600
 Wire Wire Line
-	4500 3600 4500 6250
-Wire Wire Line
-	5200 3550 5750 3550
+	4500 3600 4500 4500
 Wire Wire Line
 	6350 3550 6350 3750
@@
 L Device:R_Small R?
 U 1 1 6201D964
-P 5600 3400
+P 5550 3800
 AR Path="/60DC28BD/6201D964" Ref="R?"  Part="1"
 AR Path="/60E5E32B/6201D964" Ref="R?"  Part="1"
 AR Path="/60DB2574/60E5E32B/6201D964" Ref="R?"  Part="1"
 AR Path="/60E70F2C/60E5E32B/6201D964" Ref="R2114"  Part="1"
-F 0 "R2114" V 5700 3450 50  0000 C CNN
-F 1 "100k" V 5650 3600 50  0000 C CNN
-F 2 "Resistor_SMD:R_0603_1608Metric" H 5600 3400 50  0001 C CNN
-F 3 "~" H 5600 3400 50  0001 C CNN
-	1    5600 3400
-	0    -1   -1   0
-$EndComp
-Wire Wire Line
-	5700 3400 5750 3400
-Wire Wire Line
-	5750 3400 5750 3550
-Connection ~ 5750 3550
-Wire Wire Line
-	5750 3550 6350 3550
-Wire Wire Line
-	5500 3400 4900 3400
-Wire Wire Line
-	5200 3650 5250 3650
-Wire Wire Line
-	5250 3650 5250 3800
-Wire Wire Line
-	5250 4350 5200 4350
+F 0 "R2114" V 5650 3850 50  0000 C CNN
+F 1 "100k" V 5600 4000 50  0000 C CNN
+F 2 "Resistor_SMD:R_0603_1608Metric" H 5550 3800 50  0001 C CNN
+F 3 "~" H 5550 3800 50  0001 C CNN
+	1    5550 3800
+	0    -1   -1   0
+$EndComp
 Wire Wire Line
 	4900 3800 5250 3800
 Connection ~ 5250 3800
 Wire Wire Line
-	5250 3800 5250 4350
-Wire Wire Line
 	4900 4500 5250 4500
-Wire Wire Line
-	5250 4500 5250 4350
-Connection ~ 5250 4350
 $Comp
 L lan9254_project:GND #PWR?
@@
 $EndComp
 Wire Wire Line
-	5450 4100 4900 4100
-Connection ~ 4900 4100
-Wire Wire Line
-	5200 4250 5750 4250
-Wire Wire Line
-	5750 4250 5750 4100
-Wire Wire Line
 	5650 4100 5750 4100
 Connection ~ 5750 4100
@@
 AR Path="/60E70F2C/60E5E32B/620537D3" Ref="#PWR?"  Part="1"
 F 0 "#PWR?" H 4900 3250 50  0001 C CNN
-F 1 "+1V8" H 4915 3573 50  0000 C CNN
+F 1 "+1V8" H 4950 3550 50  0000 C CNN
 F 2 "" H 4900 3400 50  0001 C CNN
 F 3 "" H 4900 3400 50  0001 C CNN
@@
 	1    0    0    -1
 $EndComp
-Connection ~ 4900 3400
 Text HLabel 3800 700  0    50   Output ~ 0
 I2C_ISOLb
@@
 Wire Wire Line
 	6650 4400 6550 4400
-Connection ~ 6450 4400
 Wire Wire Line
 	6550 4350 6550 4400
 Connection ~ 6550 4400
-Wire Wire Line
-	6550 4400 6450 4400
 Text HLabel 10300 3150 2    50   Input ~ 0
 EEP_WP
@@
 	9900 3450 9900 3550
 Connection ~ 9900 3550
-Wire Wire Line
-	6350 3550 6350 1150
-Connection ~ 6350 3550
-Wire Wire Line
-	3800 1150 6350 1150
-Text HLabel 3800 1150 0    50   Output ~ 0
+Text HLabel 3800 4500 0    50   Output ~ 0
 EEP_SZ
+Text Notes 6100 5100 0    50   ~ 0
+RED (ErrLED)
+Text Notes 6100 6300 0    50   ~ 0
+GREEN (RunLED)
+Wire Wire Line
+	5200 4350 5750 4350
+Wire Wire Line
+	5750 4100 5750 4350
+Text Notes 5350 4750 0    50   ~ 0
+Use pin-2 input;\ncould also load\na 74LV1T04 inverter\nor a 74LV1T00 NAND
+Wire Wire Line
+	5250 3800 5250 4100
+Wire Wire Line
+	5200 4250 5200 4100
+Wire Wire Line
+	5200 4100 4900 4100
+Connection ~ 4900 4100
+Wire Wire Line
+	5450 4100 5250 4100
+Connection ~ 5250 4100
+Wire Wire Line
+	5250 4100 5250 4500
+Wire Wire Line
+	5700 3800 5700 3650
+Wire Wire Line
+	5700 3550 6350 3550
+Wire Wire Line
+	5650 3800 5700 3800
+Wire Wire Line
+	5250 3800 5450 3800
+Wire Wire Line
+	5200 3550 5200 3400
+Wire Wire Line
+	5200 3400 4900 3400
+Connection ~ 4900 3400
+Wire Wire Line
+	5200 3650 5700 3650
+Connection ~ 5700 3650
+Wire Wire Line
+	5700 3650 5700 3550
+Wire Wire Line
+	6300 4400 6550 4400
+$Comp
+L lan9254_project:+1V8 #PWR?
+U 1 1 6265E00F
+P 7200 4500
+AR Path="/60DC28BD/6265E00F" Ref="#PWR?"  Part="1"
+AR Path="/60E5E32B/6265E00F" Ref="#PWR?"  Part="1"
+AR Path="/60DB2574/60E5E32B/6265E00F" Ref="#PWR?"  Part="1"
+AR Path="/60E70F2C/60E5E32B/6265E00F" Ref="#PWR?"  Part="1"
+F 0 "#PWR?" H 7200 4350 50  0001 C CNN
+F 1 "+1V8" H 7215 4673 50  0000 C CNN
+F 2 "" H 7200 4500 50  0001 C CNN
+F 3 "" H 7200 4500 50  0001 C CNN
+	1    7200 4500
+	1    0    0    -1
+$EndComp
+Wire Wire Line
+	6350 4350 6350 4550
+Wire Wire Line
+	6350 4550 6450 4550
+Wire Wire Line
+	7200 4550 7200 4500
+Wire Wire Line
+	4600 4300 4600 5050
+Wire Wire Line
+	3800 4500 4500 4500
+Connection ~ 4500 4500
+Wire Wire Line
+	4500 4500 4500 6250
+Wire Wire Line
+	6450 4350 6450 4550
+Connection ~ 6450 4550
+Wire Wire Line
+	6450 4550 7200 4550
+$Comp
+L Device:R_Small R?
+U 1 1 62676AD9
+P 4750 3400
+AR Path="/60DC28BD/62676AD9" Ref="R?"  Part="1"
+AR Path="/60E5E32B/62676AD9" Ref="R?"  Part="1"
+AR Path="/60DB2574/60E5E32B/62676AD9" Ref="R?"  Part="1"
+AR Path="/60E70F2C/60E5E32B/62676AD9" Ref="R2116"  Part="1"
+F 0 "R2116" V 4950 3400 50  0000 C CNN
+F 1 "0" V 4850 3400 50  0000 C CNN
+F 2 "Resistor_SMD:R_0603_1608Metric" H 4750 3400 50  0001 C CNN
+F 3 "~" H 4750 3400 50  0001 C CNN
+	1    4750 3400
+	0    -1   -1   0
+$EndComp
+$Comp
+L Device:R_Small R?
+U 1 1 6267738A
+P 4750 3800
+AR Path="/60DC28BD/6267738A" Ref="R?"  Part="1"
+AR Path="/60E5E32B/6267738A" Ref="R?"  Part="1"
+AR Path="/60DB2574/60E5E32B/6267738A" Ref="R?"  Part="1"
+AR Path="/60E70F2C/60E5E32B/6267738A" Ref="R2117"  Part="1"
+F 0 "R2117" V 4950 3800 50  0000 C CNN
+F 1 "0" V 4850 3800 50  0000 C CNN
+F 2 "Resistor_SMD:R_0603_1608Metric" H 4750 3800 50  0001 C CNN
+F 3 "~" H 4750 3800 50  0001 C CNN
+	1    4750 3800
+	0    -1   1    0
+$EndComp
+Wire Wire Line
+	4650 3800 4650 3600
+Connection ~ 4650 3600
+Wire Wire Line
+	4650 3400 4650 3600
+Wire Wire Line
+	4850 3800 4900 3800
+Connection ~ 4900 3800
+Wire Wire Line
+	4850 3400 4900 3400
+Text Notes 5050 3400 0    50   ~ 0
+Instead of U2105\nR2116 OR R2117\njumpers could be loaded.
 $EndSCHEMATC
