File: IO_driver.kicad_sch (KiCad schematic)
At the start: 9 parts, among them J2002 IO_CONN, U2002 74LVC2T45DC

Commit message: WIP
Parts:
- renumbered C2003 to C2001, C2004 to C2002, J2002 to J2001, R2006 to R2001, R2007 to R2002, R2008 to R2003, R2009 to R2004, R2010 to R2005, U2002 to U2001
