File: lan9254.kicad_sch (KiCad schematic)
At the start: 42 parts, among them U18 74LVC1T126, U2301 lan9254, X2301 FNETHE025

Commit message: WIP
Parts:
- removed R2305: 0, Resistor_SMD:R_0603_1608Metric, symbol Device:R_Small
- removed R2306: 10k, Resistor_SMD:R_0603_1608Metric, symbol Device:R_Small
- added TP2306: GND, Connector_PinHeader_2.54mm:PinHeader_1x01_P2.54mm_Vertical, symbol Connector:TestPoint
- TP2301, TP2302, TP2303, TP2304, TP2305: footprint Connector_PinHeader_1.27mm:PinHeader_1x01_P1.27mm_Vertical -> Connector_PinHeader_2.54mm:PinHeader_1x01_P2.54mm_Vertical
Connections:
- net GND_lan9254: now also TP2306.1
Other:
- removed sheet IO_driver_2
- removed sheet IO_driver_3
- removed sheet lan9254_jtag
- note removed: "(In case buffer is not loaded omitting R2305 makes FPGA-JTAG independent of TESTMODE)"
